Commit message: added stls and node can access the stl data

File: camera_viewpoint_selection_algorithms/info_entropy/urdfs/box.urdf (robot description, URDF)
Before this commit: robot box, 1 links, 0 joints
Links:
- link box: geometry collision mesh filename=package://info_entropy/urdfs/cube.STL scale=.001 .001 .001; visual mesh filename=package://info_entropy/urdfs/cube.STL scale=.001 .001 .001

Commit message: added stls and node can access the stl data rviz launches with box

File: camera_viewpoint_selection_algorithms/info_entropy/urdfs/box.urdf (robot description, URDF)
Before this commit: robot box, 1 links, 0 joints
Links:
- link box: geometry collision mesh filename=package://info_entropy/urdfs/box.STL scale=.01 .01 .01; visual mesh filename=package://info_entropy/urdfs/box.STL scale=.01 .01 .01

Commit message: one launch file to rule them all

File: camera_viewpoint_selection_algorithms/info_entropy/urdfs/box.urdf (robot description, URDF)
Before this commit: robot box, 1 links, 0 joints
Links:
- link box: mass 1.0 -> 0

Commit message: box moves in gazebo and info knows where camera is

File: camera_viewpoint_selection_algorithms/info_entropy/urdfs/box.urdf (robot description, URDF)
Before this commit: robot box, 1 links, 0 joints
Links:
- link box: mass 0 -> 0.001
